File: KiCAD/Sunflower.kicad_pcb (KiCad board)
At the start: 2 copper layers, 100 x 100 mm, 18 parts, among them J1 Banana 4mm, J10 Banana 4mm, J11 Banana 4mm, J12 Banana 4mm, J13 Banana 4mm, J14 Banana 4mm, J15 Banana 4mm, J16 Banana 4mm, J2 Banana 4mm, J3 Banana 4mm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

Commit message: Uploaded Sunflower v2
Adds thermal pads
Routing:
- added copper zone on F.Cu, net GND
Other:
- board text added: "Sunflower v2 JPC-12 radials disk"
- board text removed: "Sunflower JPC-12 radials disk"
